Commit message: general update

File: assets/urdf/robotiq_arg85_description/robots/robotiq_arg85_description.urdf (robot description, URDF)
Before this commit: robot robotiq_arg85_description, 22 links, 21 joints
Links:
- removed link rev_link1
- removed link rev_link2
- removed link rev_link3
- removed link rev_link_twist
- removed link slide_x
- removed link slide_y
- removed link slide_z
Joints:
- removed joint rev_joint1
- removed joint rev_joint2
- removed joint rev_joint3
- removed joint rev_twist
- removed joint slide_jointx
- removed joint slide_jointy
- removed joint slide_jointz
- joint rev_jointx: child rev_link_twist -> robotiq_85_base_link
